File: design files/Din25 Ver/rascsi_din.sch (EAGLE design)
At the start: 16 parts, among them U11 SN74LS641-1SC, U22 SN74LS641-1SC, U33 SN74LS641-1SC, U44 SN74LS641-1SC, X1 2550-

Commit message: New boards
Shrunk internal board down to min size. Also added a din25 board for external use.
Parts:
- removed J1: (no value), con-amp:FLOP-4W
- added JP1: (no value), pinhead:PINHD-1X2
- X1: value 2550- -> (none); device con-3m:2550- -> con-subd:F25HPS
Connections:
- removed net +12V: J1.1
- net +3V3: no longer U$1.3V3@1
- net +5V: no longer J1.4
- net ACK: now also RN1.3; no longer RN1.8
- net ACT: now also JP1.1
- net ATN: now also RN1.2; no longer RN1.7
- net BSY: now also RN1.6; no longer RN1.2
- net C-ACK: now also X1-5.F; no longer X1-38.KL
- net C-ATN: now also X1-17.F; no longer X1-32.KL
- net C-BSY: now also X1-6.F; no longer X1-36.KL
- net C-CD: now also X1-15.F; no longer X1-46.KL
- net C-D0: now also X1-8.F; no longer X1-2.KL
- net C-D1: now also X1-21.F; no longer X1-4.KL
- net C-D2: now also X1-22.F; no longer X1-6.KL
- net C-D3: now also X1-10.F; no longer X1-8.KL
- net C-D4: now also X1-23.F; no longer X1-10.KL
- net C-D5: now also X1-11.F; no longer X1-12.KL
- net C-D6: now also X1-12.F; no longer X1-14.KL
- net C-D7: now also X1-13.F; no longer X1-16.KL
- net C-DP: now also X1-20.F; no longer X1-18.KL
- net C-IO: now also X1-3.F; no longer X1-50.KL
- net C-MSG: now also X1-2.F; no longer X1-42.KL
- net C-REQ: now also X1-1.F; no longer X1-48.KL
- net C-RST: now also X1-4.F; no longer X1-40.KL
- net C-SEL: now also X1-19.F; no longer X1-44.KL
- net CD: now also RN1.8; no longer RN1.4
- net GND: now also JP1.2, X1-14.F, X1-16.F, X1-18.F, X1-24.F, X1-7.F, X1-9.F; no longer J1.2, J1.3, X1-20.KL, X1-22.KL, X1-24.KL, X1-28.KL, X1-30.KL, X1-34.KL
- net IO: now also RN1.10; no longer RN1.6
- net MSG: now also RN1.7; no longer RN1.3
- net REQ: now also RN1.9; no longer RN1.5
- net RST: now also RN1.4; no longer RN1.9
- net SEL: now also RN1.5; no longer RN1.10
- net TERMPOW: now also X1-25.F; no longer X1-26.KL
Other:
- moved on the sheet: X1-1, X1-10, X1-11, X1-12, X1-13, X1-14, X1-15, X1-16, X1-17, X1-18, X1-19, X1-2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
